File: Eagle/mwscoretransponder2017.brd (EAGLE design)
At the start: 44.5 x 44.5 mm, 36 parts, among them J1 ISP, J10 5267-3, J2 5267-3, J6 5267-3, J7 5267-3, J8 5267-3, J9 5267-3, U1 ATMEGA168, U2 MIC5219 5V, U3 MIC5219 3.3V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

Commit message: Minor Updates
Minor Updates
Parts:
- C11: value 470pf -> 470pF
- C12, C3: value (none) -> 2.2uF
- C6: value 100nF -> 0.1uF
- moved R1 0.76 mm to (39.4, 37.8), turned to 270 degrees
Routing:
- net 5V: track 156.3 -> 155.5 mm
- net RESET: track 55.5 -> 56.0 mm
Changed lines of the file:
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@@
 <setting verticaltext="up"/>
 </settings>
-<grid distance="0.01" unitdist="inch" unit="mil" style="lines" multiple="1" display="no" altdistance="0.025" altunitdist="inch" altunit="inch"/>
+<grid distance="1" unitdist="mil" unit="mil" style="lines" multiple="1" display="no" altdistance="0.025" altunitdist="inch" altunit="inch"/>
 <layers>
 <layer number="1" name="Top" color="4" fill="1" visible="yes" active="yes"/>
@@
 <wire x1="34.08400625" y1="42.588003125" x2="35.00399375" y2="42.588003125" width="0.2032" layer="121"/>
 <text x="33.8455" y="41.275" size="0.6096" layer="121" font="vector" rot="R90">PWR</text>
-<text x="40.005" y="36.83" size="0.6096" layer="121" font="vector" rot="R180">R1</text>
+<text x="40.1066" y="40.1828" size="0.6096" layer="121" font="vector" rot="R180">R1</text>
 <text x="35.179" y="37.338" size="0.6096" layer="121" font="vector" rot="R180">R2</text>
 <text x="37.719" y="37.338" size="0.6096" layer="121" font="vector" rot="R180">R3</text>
@@
 <element name="U1" library="SparkFun" package="TQFP32-08" value="ATMEGA168" x="26.67" y="22.606" rot="R270"/>
 <element name="S1" library="smd-special" package="SMS-008" value="SWS008" x="25.4" y="7.112"/>
-<element name="R1" library="SparkFun" package="0603-RES" value="10k" x="39.37" y="38.608" rot="R90"/>
+<element name="R1" library="SparkFun" package="0603-RES" value="10k" x="39.37" y="37.846" rot="R270"/>
 <element name="R2" library="SparkFun" package="0603-RES" value="1k" x="34.544" y="39.116" rot="R90"/>
 <element name="R3" library="SparkFun" package="0603-RES" value="1k" x="37.084" y="39.116" rot="R90"/>
@@
 <element name="Y1" library="SparkFun" package="CRYSTAL-SMD-5X3" value="" x="24.892" y="30.734" rot="R180"/>
 <element name="J5" library="SparkFun" package="1X06" value="" x="41.91" y="22.86" rot="R90"/>
-<element name="C6" library="SparkFun" package="0603-CAP" value="100nF" x="42.418" y="38.1" rot="R180"/>
+<element name="C6" library="SparkFun" package="0603-CAP" value="0.1uF" x="42.418" y="38.1" rot="R180"/>
 <element name="R12" library="SparkFun" package="0603-RES" value="1k" x="18.796" y="23.368" rot="MR0"/>
 <element name="R13" library="SparkFun" package="0603-RES" value="1k" x="18.796" y="25.908" rot="MR0"/>
@@
 <element name="C2" library="rcl" package="C0603" value="470pF" x="16.256" y="36.576" rot="R180"/>
 <element name="C10" library="rcl" package="C0603" value="1uF" x="24.638" y="40.894" rot="R270"/>
-<element name="C11" library="rcl" package="C0603" value="470pf" x="25.908" y="36.576" rot="R180"/>
+<element name="C11" library="rcl" package="C0603" value="470pF" x="25.908" y="36.576" rot="R180"/>
 <element name="C13" library="SparkFun" package="0603-CAP" value="0.1uF" x="23.622" y="15.494" rot="MR0"/>
-<element name="C3" library="rcl" package="C0805" value="" x="21.59" y="40.132" rot="R90"/>
-<element name="C12" library="rcl" package="C0805" value="" x="31.242" y="39.878" rot="R90"/>
+<element name="C3" library="rcl" package="C0805" value="2.2uF" x="21.59" y="40.132" rot="R90"/>
+<element name="C12" library="rcl" package="C0805" value="2.2uF" x="31.242" y="39.878" rot="R90"/>
 </elements>
 <signals>
@@
 <wire x1="26.924" y1="27.0446" x2="27.07" y2="26.8986" width="0.254" layer="1"/>
 <wire x1="35.814" y1="38.4048" x2="34.5948" y2="38.4048" width="0.1524" layer="1"/>
-<wire x1="36.576" y1="39.1668" x2="35.814" y2="38.4048" width="0.1524" layer="1"/>
-<wire x1="38.3032" y1="39.1668" x2="36.576" y2="39.1668" width="0.1524" layer="1"/>
-<wire x1="38.8112" y1="37.8968" x2="38.3032" y2="39.1668" width="0.1524" layer="1"/>
+<wire x1="35.814" y1="38.4048" x2="36.5506" y2="39.116" width="0.1524" layer="1"/>
 <wire x1="34.5948" y1="38.4048" x2="34.544" y2="38.266" width="0.1524" layer="1"/>
-<wire x1="38.8112" y1="37.8968" x2="39.37" y2="37.758" width="0.1524" layer="1"/>
 <wire x1="21.1836" y1="38.862" x2="19.3548" y2="38.862" width="0.1524" layer="1"/>
 <wire x1="21.4884" y1="39.1668" x2="21.1836" y2="38.862" width="0.1524" layer="1"/>
@@
 <wire x1="19.2024" y1="38.862" x2="19.238" y2="38.8319" width="0.1524" layer="1"/>
 <wire x1="5.334" y1="25.146" x2="5.294" y2="25.146" width="0.1524" layer="1"/>
+<wire x1="36.5506" y1="39.116" x2="38.793990625" y2="39.116" width="0.1524" layer="1"/>
+<wire x1="38.793990625" y1="39.116" x2="38.97359375" y2="39.04160625" width="0.1524" layer="1" curve="-44.999502"/>
+<wire x1="38.97359375" y1="39.04160625" x2="39.37" y2="38.696" width="0.1524" layer="1"/>
 </signal>
 <signal name="RESET">
@@
 <contactref element="R1" pad="2"/>
 <contactref element="C6" pad="2"/>
-<wire x1="41.3004" y1="38.1" x2="39.9796" y2="39.4208" width="0.1524" layer="1"/>
-<wire x1="39.9796" y1="39.4208" x2="39.37" y2="39.458" width="0.1524" layer="1"/>
 <wire x1="32.6136" y1="22.86" x2="31.0896" y2="22.86" width="0.1524" layer="1"/>
 <wire x1="33.8328" y1="22.86" x2="32.6136" y2="22.86" width="0.1524" layer="16"/>
@@
 <wire x1="40.0812" y1="13.1064" x2="40.0812" y2="17.3736" width="0.1524" layer="1"/>
 <wire x1="41.91" y1="11.2776" x2="40.0812" y2="13.1064" width="0.1524" layer="1"/>
-<wire x1="41.4528" y1="38.1" x2="41.3004" y2="38.1" width="0.1524" layer="1"/>
-<wire x1="41.4528" y1="38.1" x2="41.568" y2="38.1" width="0.1524" layer="1"/>
+<wire x1="41.568" y1="38.1" x2="41.3004" y2="38.1" width="0.1524" layer="1"/>
 <wire x1="41.91" y1="11.2776" x2="41.91" y2="11.176" width="0.1524" layer="1"/>
 <via x="32.6136" y="22.86" extent="1-16" drill="0.3048"/>
+<wire x1="39.37" y1="36.996" x2="39.964190625" y2="36.996" width="0.1524" layer="1"/>
+<wire x1="39.964190625" y1="36.996" x2="40.14379375" y2="37.07039375" width="0.1524" layer="1" curve="44.999502"/>
+<wire x1="40.14379375" y1="37.07039375" x2="40.4114" y2="37.338" width="0.1524" layer="1"/>
+<wire x1="40.4114" y1="37.338" x2="40.4114" y2="37.816990625" width="0.1524" layer="1"/>
+<wire x1="40.4114" y1="37.816990625" x2="40.48579375" y2="37.99659375" width="0.1524" layer="1" curve="-44.999502"/>
+<wire x1="40.48579375" y1="37.99659375" x2="40.6146" y2="38.1254" width="0.1524" layer="1"/>
+<wire x1="40.6146" y1="38.1254" x2="41.506678125" y2="38.1254" width="0.1524" layer="1"/>
+<wire x1="41.506678125" y1="38.1254" x2="41.568" y2="38.1" width="0.254" layer="1" curve="-45"/>
 </signal>
 <signal name="MISO">
