File: Eagle/mwscoretransponder2017.sch (EAGLE design)
At the start: 36 parts, among them J1 ISP, J10 5267-3, J2 5267-3, J6 5267-3, J7 5267-3, J8 5267-3, J9 5267-3, U1 ATMEGA168, U2 MIC5219 5V, U3 MIC5219 3.3V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

Commit message: Minor Updates
Minor Updates
Parts:
- C11: value 470pf -> 470pF
- C12, C3: value (none) -> 2.2uF
- C6: value 100nF -> 0.1uF
Changed lines of the file:
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@@
 <?xml version="1.0" encoding="utf-8"?>
 <!DOCTYPE eagle SYSTEM "eagle.dtd">
-<eagle version="7.6.0">
+<eagle version="8.0.1">
 <drawing>
 <settings>
@@
 <part name="P+1" library="SparkFun" deviceset="VCC" device=""/>
 <part name="J5" library="SparkFun" deviceset="M06" device="SIP"/>
-<part name="C6" library="SparkFun" deviceset="CAP" device="0603-CAP" value="100nF"/>
+<part name="C6" library="SparkFun" deviceset="CAP" device="0603-CAP" value="0.1uF"/>
 <part name="GND10" library="SparkFun" deviceset="GND" device=""/>
 <part name="U$1" library="SparkFun" deviceset="5V" device=""/>
@@
 <part name="C2" library="rcl" deviceset="C-US" device="C0603" value="470pF"/>
 <part name="C10" library="rcl" deviceset="C-US" device="C0603" value="1uF"/>
-<part name="C11" library="rcl" deviceset="C-US" device="C0603" value="470pf"/>
+<part name="C11" library="rcl" deviceset="C-US" device="C0603" value="470pF"/>
 <part name="C13" library="SparkFun" deviceset="CAP" device="0603-CAP" value="0.1uF"/>
-<part name="C3" library="rcl" deviceset="C-US" device="C0805"/>
-<part name="C12" library="rcl" deviceset="C-US" device="C0805"/>
+<part name="C3" library="rcl" deviceset="C-US" device="C0805" value="2.2uF"/>
+<part name="C12" library="rcl" deviceset="C-US" device="C0805" value="2.2uF"/>
 </parts>
 <sheets>
